File: stella-1.2-permaproto-replacement/stella-1.2-permaproto-replacement.kicad_sch (KiCad schematic)
At the start: 14 parts, among them J1 Conn_01x03, J2 Conn_01x04, SW1 RotaryEncoder_Switch, SW2 SW_Push, U1 Eyespi Breakout, U2 RTC, U3 MiniBoost, U4 GPS Breakout, U5 SD Reader

Commit message: Finalize v0.1.0 of base pcb
Connections:
- net at R1.1, U3.4 (EN): now also A1.22 (A9/IO33); no longer A1.23 (A10/IO27)
- net at U1.7 (TFTDC): now also A1.23 (A10/IO27); no longer A1.24 (A11/IO12)
- net at U1.9 (TCS): now also A1.24 (A11/IO12); no longer A1.25 (A12/IO13)
- net at A1.8 (I39/A3): now also SW1.B; no longer SW1.A
- net at A1.9 (IO36/A4): now also SW1.A; no longer SW1.B
Changed lines of the file:
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@@
+	)
+	(no_connect
+		(at 124.46 88.9)
 	)
 	(no_connect
@@
 	)
 	(no_connect
-		(at 124.46 81.28)
-	)
-	(no_connect
 		(at 181.61 137.16)
 	)
@@
 	(wire
 		(pts
-			(xy 212.09 107.95) (xy 198.12 107.95)
+			(xy 91.44 86.36) (xy 91.44 82.55)
 		)
 		(stroke
@@
 	(wire
 		(pts
+			(xy 105.41 81.28) (xy 124.46 81.28)
+		)
+		(stroke
+			(width 0)
+			(type default)
+		)
+	)
+	(wire
+		(pts
 			(xy 149.86 93.98) (xy 191.77 93.98)
 		)
@@
 	(wire
 		(pts
-			(xy 124.46 88.9) (xy 78.74 88.9)
-		)
-		(stroke
-			(width 0)
-			(type default)
-		)
-	)
-	(wire
-		(pts
 			(xy 158.75 57.15) (xy 166.37 57.15)
 		)
@@
 	(wire
 		(pts
-			(xy 67.31 86.36) (xy 67.31 87.63)
+			(xy 105.41 81.28) (xy 105.41 66.04)
 		)
 		(stroke
@@
 	(wire
 		(pts
-			(xy 124.46 83.82) (xy 105.41 83.82)
-		)
-		(stroke
-			(width 0)
-			(type default)
-		)
-	)
-	(wire
-		(pts
 			(xy 114.3 99.06) (xy 124.46 99.06)
 		)
@@
 	(wire
 		(pts
+			(xy 207.01 100.33) (xy 198.12 100.33)
+		)
+		(stroke
+			(width 0)
+			(type default)
+		)
+	)
+	(wire
+		(pts
 			(xy 73.66 55.88) (xy 80.01 55.88)
 		)
@@
 	(wire
 		(pts
+			(xy 91.44 82.55) (xy 67.31 82.55)
+		)
+		(stroke
+			(width 0)
+			(type default)
+		)
+	)
+	(wire
+		(pts
 			(xy 102.87 58.42) (xy 102.87 67.31)
 		)
@@
 	(wire
 		(pts
-			(xy 203.2 100.33) (xy 207.01 100.33)
-		)
-		(stroke
-			(width 0)
-			(type default)
-		)
-	)
-	(wire
-		(pts
-			(xy 78.74 82.55) (xy 67.31 82.55)
-		)
-		(stroke
-			(width 0)
-			(type default)
-		)
-	)
-	(wire
-		(pts
 			(xy 191.77 93.98) (xy 191.77 85.09)
 		)
@@
 	(wire
 		(pts
-			(xy 78.74 88.9) (xy 78.74 82.55)
-		)
-		(stroke
-			(width 0)
-			(type default)
-		)
-	)
-	(wire
-		(pts
-			(xy 198.12 107.95) (xy 198.12 99.06)
+			(xy 198.12 99.06) (xy 198.12 100.33)
+		)
+		(stroke
+			(width 0)
+			(type default)
+		)
+	)
+	(wire
+		(pts
+			(xy 76.2 87.63) (xy 67.31 87.63)
 		)
 		(stroke
@@
 	(wire
 		(pts
-			(xy 212.09 100.33) (xy 212.09 107.95)
-		)
-		(stroke
-			(width 0)
-			(type default)
-		)
-	)
-	(wire
-		(pts
 			(xy 73.66 53.34) (xy 80.01 53.34)
 		)
@@
 	(wire
 		(pts
+			(xy 203.2 104.14) (xy 212.09 104.14)
+		)
+		(stroke
+			(width 0)
+			(type default)
+		)
+	)
+	(wire
+		(pts
 			(xy 191.77 121.92) (xy 191.77 137.16)
 		)
@@
 	(wire
 		(pts
+			(xy 212.09 104.14) (xy 212.09 100.33)
+		)
+		(stroke
+			(width 0)
+			(type default)
+		)
+	)
+	(wire
+		(pts
 			(xy 175.26 80.01) (xy 175.26 83.82)
 		)
@@
 	(wire
 		(pts
-			(xy 203.2 96.52) (xy 203.2 100.33)
+			(xy 203.2 96.52) (xy 203.2 104.14)
 		)
 		(stroke
@@
 	(wire
 		(pts
+			(xy 124.46 86.36) (xy 91.44 86.36)
+		)
+		(stroke
+			(width 0)
+			(type default)
+		)
+	)
+	(wire
+		(pts
 			(xy 172.72 80.01) (xy 172.72 88.9)
 		)
@@
 	(wire
 		(pts
-			(xy 124.46 86.36) (xy 67.31 86.36)
-		)
-		(stroke
-			(width 0)
-			(type default)
-		)
-	)
-	(wire
-		(pts
 			(xy 158.75 54.61) (xy 166.37 54.61)
 		)
@@
 	(wire
 		(pts
+			(xy 76.2 83.82) (xy 124.46 83.82)
+		)
+		(stroke
+			(width 0)
+			(type default)
+		)
+	)
+	(wire
+		(pts
 			(xy 96.52 106.68) (xy 101.6 106.68)
 		)
@@
 	(wire
 		(pts
-			(xy 105.41 83.82) (xy 105.41 66.04)
-		)
-		(stroke
-			(width 0)
-			(type default)
-		)
-	)
-	(wire
-		(pts
 			(xy 186.69 68.58) (xy 195.58 68.58)
 		)
@@
 		)
 		(stroke
+			(width 0)
+			(type default)
+		)
+	)
+	(wire
+		(pts
+			(xy 76.2 83.82) (xy 76.2 87.63)
+		)
+		(stroke
