File: stella-1.2-rs-permaproto-replacement/stella-1.2-rs-permaproto-replacement.kicad_pcb (KiCad board)
At the start: 2 copper layers, 81.3 x 50.8 mm, 10 parts, among them J1 Conn_01x03, J2 Conn_01x04, U1 Triad, U2 Humidity, U3 Surface Temp, U4 Range

Commit message: Update gerbers with silkscreen info
Other:
- board text added: "STELLA-1.2 Remote Sensing Permaproto Replacement PCB v0.1.1 2026 Layout by Nathan Eloe Should line up with original permaproto component placement"
- board text removed: "Stella-1.2 Remote Sensing Permaproto Replacement PCB v0.1.1 2026 Layout by Nathan Eloe Should line up with original permaproto component placement"
Changed lines of the file:
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@@
 		)
 	)
-	(gr_text "Stella-1.2 Remote Sensing Permaproto Replacement PCB v0.1.1\n2026\nLayout by Nathan Eloe\nShould line up with original permaproto component placement"
+	(gr_text "STELLA-1.2 Remote Sensing Permaproto Replacement PCB v0.1.1\n2026\nLayout by Nathan Eloe\nShould line up with original permaproto component placement"
 		(at 107 125 0)
 		(layer "F.SilkS")

Commit message: Add Paul M attribution for NASA Stella
Other:
- board text added: "STELLA-1.2 Remote Sensing Permaproto Replacement PCB v0.1.1 2026 NASA STELLA-1.2 created by Paul Mirel PCBLayout by Nathan Eloe"
- board text removed: "STELLA-1.2 Remote Sensing Permaproto Replacement PCB v0.1.1 2026 Layout by Nathan Eloe Should line up with original permaproto component placement"
Changed lines of the file:
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@@
 		)
 	)
-	(gr_text "STELLA-1.2 Remote Sensing Permaproto Replacement PCB v0.1.1\n2026\nLayout by Nathan Eloe\nShould line up with original permaproto component placement"
+	(gr_text "STELLA-1.2 Remote Sensing Permaproto Replacement PCB v0.1.1\n2026\nNASA STELLA-1.2 created by Paul Mirel\nPCBLayout by Nathan Eloe\n"
 		(at 107 125 0)
 		(layer "F.SilkS")
