File: stella-1.2-base/stella-1.2-permaproto-replacement.kicad_pcb (KiCad board)
At the start: 2 copper layers, 157.5 x 50.8 mm, 15 parts, among them J1 Conn_01x03, J2 Conn_01x04, SW1 RotaryEncoder_Switch, SW2 SW_Push, U1 Eyespi Breakout, U2 RTC, U3 MiniBoost, U4 GPS Breakout, U5 SD Reader

Commit message: Clean up silkscreens on base pcb
Other:
- board text added: "Flat Coupler Jig"
- board text added: "POPO Switch"
- board text added: "Rotary Encoder"
- board text added: "STELLA-1.2 Base PCB v0.1.1 2026 STELLA-1.2 created by Paul Mirel, NASA Goddard PCB Layout by Nathan Eloe, Northwest Missouri State University"
- board text removed: "STELLA-1.2 Base Permaproto Replacement PCB v0.1.1 2026 NASA STELLA-1.2 created by Paul Mirel PCB Layout by Nathan Eloe"
Changed lines of the file:
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@@
 			(at 2.42 0.07 90)
 			(layer "F.SilkS")
+			(hide yes)
 			(effects
 				(font
@@
 			(unlocked yes)
 			(layer "F.SilkS")
+			(hide yes)
 			(effects
 				(font
@@
 		(property "Value" "10k"
 			(at 3.81 1.92 90)
-			(layer "F.Fab")
+			(layer "F.SilkS")
 			(effects
 				(font
@@
 			(unlocked yes)
 			(layer "F.SilkS")
+			(hide yes)
 			(effects
 				(font
@@
 		)
 		(property "Value" ".1uF"
-			(at 1.25 4.4 0)
-			(layer "F.Fab")
+			(at -3.52 0.02 180)
+			(layer "F.SilkS")
 			(effects
 				(font
@@
 			(unlocked yes)
 			(layer "F.SilkS")
+			(hide yes)
 			(effects
 				(font
@@
 			(unlocked yes)
 			(layer "F.SilkS")
+			(hide yes)
 			(effects
 				(font
@@
 			(unlocked yes)
 			(layer "F.SilkS")
+			(hide yes)
 			(effects
 				(font
@@
 		(property "Value" "10k"
 			(at 3.81 1.92 90)
-			(layer "F.Fab")
+			(layer "F.SilkS")
 			(effects
 				(font
@@
 		(property "Value" "10k"
 			(at 3.81 1.92 90)
-			(layer "F.Fab")
+			(layer "F.SilkS")
 			(effects
 				(font
@@
 			(unlocked yes)
 			(layer "B.SilkS")
+			(hide yes)
 			(effects
 				(font
@@
 			(at 3 4.75 90)
 			(layer "B.SilkS")
+			(hide yes)
 			(effects
 				(font
@@
 		)
 	)
+	(gr_text "Flat Coupler Jig"
+		(at 87 100.53 90)
+		(layer "F.SilkS")
+		(effects
+			(font
+				(size 1 1)
+				(thickness 0.1)
+			)
+			(justify bottom)
+		)
+	)
 	(gr_text "Vin"
 		(at 89.916 114.554 0)
@@
 		)
 	)
-	(gr_text "STELLA-1.2 Base Permaproto Replacement PCB v0.1.1\n2026\nNASA STELLA-1.2 created by Paul Mirel\nPCB Layout by Nathan Eloe"
-		(at 229.5 84 0)
+	(gr_text "POPO Switch"
+		(at 202.5 119.5 0)
 		(layer "B.SilkS")
 		(effects
@@
 		)
 	)
+	(gr_text "Rotary\nEncoder"
+		(at 177.5 99.5 0)
+		(layer "B.SilkS")
+		(effects
+			(font
+				(size 1 1)
+				(thickness 0.1)
+			)
+			(justify bottom mirror)
+		)
+	)
 	(gr_text "A1\nAdafruit 5447\nESP32-S3 Feather, 4MB Flash 2MB PSRAM\nLong pins through Feather"
 		(at 212.5 102.945 0)
@@
 		)
 	)
+	(gr_text "STELLA-1.2 Base PCB v0.1.1\n2026\nSTELLA-1.2 created by Paul Mirel, NASA Goddard\nPCB Layout by Nathan Eloe, Northwest Missouri State University"
+		(at 229.5 86 0)
+		(layer "B.SilkS")
+		(effects
+			(font
+				(size 1.5 1.5)
+				(thickness 0.15)
+			)
+			(justify left bottom mirror)
+		)
+	)

Commit message: Tighten attribution to 3 lines
Other:
- board text added: "STELLA-1.2 Base PCB v0.1.1, 2026 STELLA-1.2 created by Paul Mirel, NASA Goddard PCB Layout by Nathan Eloe, Northwest Missouri State University"
- board text removed: "STELLA-1.2 Base PCB v0.1.1 2026 STELLA-1.2 created by Paul Mirel, NASA Goddard PCB Layout by Nathan Eloe, Northwest Missouri State University"
Changed lines of the file:
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@@
 		)
 	)
-	(gr_text "STELLA-1.2 Base PCB v0.1.1\n2026\nSTELLA-1.2 created by Paul Mirel, NASA Goddard\nPCB Layout by Nathan Eloe, Northwest Missouri State University"
-		(at 229.5 86 0)
+	(gr_text "STELLA-1.2 Base PCB v0.1.1, 2026\nSTELLA-1.2 created by Paul Mirel, NASA Goddard\nPCB Layout by Nathan Eloe, Northwest Missouri State University"
+		(at 229.5 85 0)
 		(layer "B.SilkS")
 		(effects

Commit message: Remove unneeded schematic refs from silkscreen
Other:
- board text added: "Adafruit 5447 ESP32-S3 Feather, 4MB Flash 2MB PSRAM Long pins through Feather"
- board text removed: "A1 Adafruit 5447 ESP32-S3 Feather, 4MB Flash 2MB PSRAM Long pins through Feather"
Changed lines of the file:
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@@
 			(at 10.16 7.62 90)
 			(layer "B.SilkS")
+			(hide yes)
 			(effects
 				(font
@@
 			(unlocked yes)
 			(layer "B.SilkS")
+			(hide yes)
 			(effects
 				(font
@@
 			(unlocked yes)
 			(layer "B.SilkS")
+			(hide yes)
 			(effects
 				(font
@@
 		)
 	)
-	(gr_text "A1\nAdafruit 5447\nESP32-S3 Feather, 4MB Flash 2MB PSRAM\nLong pins through Feather"
-		(at 212.5 102.945 0)
+	(gr_text "Adafruit 5447\nESP32-S3 Feather, 4MB Flash 2MB PSRAM\nLong pins through Feather"
+		(at 212.5 101.5 0)
 		(layer "B.SilkS")
 		(effects
